File: TILE_0102/TILE_0102.kicad_sch (KiCad schematic)
At the start: 3 parts

Commit message: New design
Parts:
- removed H1, H2, H3: MountingHole, MountingHole:MountingHole_2.2mm_M2, symbol Mechanical:MountingHole
Changed lines of the file:
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@@
     (title "#0102")
-  )
-  (symbol (lib_id "Mechanical:MountingHole") (at 25.4 177.8 0) (unit 1)
-    (in_bom yes) (on_board yes)
-    (property "Reference" "H1" (id 0) (at 27.94 176.6316 0)
-      (effects (font (size 1.27 1.27)) (justify left))
-    )
-    (property "Value" "MountingHole" (id 1) (at 27.94 178.943 0)
-      (effects (font (size 1.27 1.27)) (justify left))
-    )
-    (property "Footprint" "MountingHole:MountingHole_2.2mm_M2" (id 2) (at 25.4 177.8 0)
-      (effects (font (size 1.27 1.27)) hide)
-    )
-    (property "Datasheet" "~" (id 3) (at 25.4 177.8 0)
-      (effects (font (size 1.27 1.27)) hide)
-    )
-    (property "Manufacturer" "~" (id 4) (at 25.4 177.8 0)
-      (effects (font (size 1.27 1.27)) hide)
-    )
-    (property "PartNumber" "~" (id 5) (at 25.4 177.8 0)
-      (effects (font (size 1.27 1.27)) hide)
-    )
-    (property "Supplier" "~" (id 6) (at 25.4 177.8 0)
-      (effects (font (size 1.27 1.27)) hide)
-    )
-  )
-  (symbol (lib_id "Mechanical:MountingHole") (at 25.4 182.88 0) (unit 1)
-    (in_bom yes) (on_board yes)
-    (property "Reference" "H2" (id 0) (at 27.94 181.7116 0)
-      (effects (font (size 1.27 1.27)) (justify left))
-    )
-    (property "Value" "MountingHole" (id 1) (at 27.94 184.023 0)
-      (effects (font (size 1.27 1.27)) (justify left))
-    )
-    (property "Footprint" "MountingHole:MountingHole_2.2mm_M2" (id 2) (at 25.4 182.88 0)
-      (effects (font (size 1.27 1.27)) hide)
-    )
-    (property "Datasheet" "~" (id 3) (at 25.4 182.88 0)
-      (effects (font (size 1.27 1.27)) hide)
-    )
-    (property "Manufacturer" "~" (id 4) (at 25.4 182.88 0)
-      (effects (font (size 1.27 1.27)) hide)
-    )
-    (property "PartNumber" "~" (id 5) (at 25.4 182.88 0)
-      (effects (font (size 1.27 1.27)) hide)
-    )
-    (property "Supplier" "~" (id 6) (at 25.4 182.88 0)
-      (effects (font (size 1.27 1.27)) hide)
-    )
-  )
-  (symbol (lib_id "Mechanical:MountingHole") (at 25.4 187.96 0) (unit 1)
-    (in_bom yes) (on_board yes)
-    (property "Reference" "H3" (id 0) (at 27.94 186.7916 0)
-      (effects (font (size 1.27 1.27)) (justify left))
-    )
-    (property "Value" "MountingHole" (id 1) (at 27.94 189.103 0)
-      (effects (font (size 1.27 1.27)) (justify left))
-    )
-    (property "Footprint" "MountingHole:MountingHole_2.2mm_M2" (id 2) (at 25.4 187.96 0)
-      (effects (font (size 1.27 1.27)) hide)
-    )
-    (property "Datasheet" "~" (id 3) (at 25.4 187.96 0)
-      (effects (font (size 1.27 1.27)) hide)
-    )
-    (property "Manufacturer" "~" (id 4) (at 25.4 187.96 0)
-      (effects (font (size 1.27 1.27)) hide)
-    )
-    (property "PartNumber" "~" (id 5) (at 25.4 187.96 0)
-      (effects (font (size 1.27 1.27)) hide)
-    )
-    (property "Supplier" "~" (id 6) (at 25.4 187.96 0)
-      (effects (font (size 1.27 1.27)) hide)
-    )
   )
   (sheet_instances
     (path "/" (page "1"))
   )
-  (symbol_instances
-    (path "/00000000-0000-0000-0000-000063082217"
-      (reference "H1") (unit 1) (value "MountingHole") (footprint "MountingHole:MountingHole_2.2mm_M2")
-    )
-    (path "/00000000-0000-0000-0000-0000630827a3"
-      (reference "H2") (unit 1) (value "MountingHole") (footprint "MountingHole:MountingHole_2.2mm_M2")
-    )
-    (path "/00000000-0000-0000-0000-000063089fe0"
-      (reference "H3") (unit 1) (value "MountingHole") (footprint "MountingHole:MountingHole_2.2mm_M2")
-    )
-  )
 )
