File: TILE_0102/TILE_0102.kicad_pcb (KiCad board)
At the start: 2 copper layers, 42.1 x 24.6 mm, 3 parts

Commit message: New design
Parts:
- removed H1, H2, H3: MountingHole, MountingHole:MountingHole_2.2mm_M2
- added kibuzzard-631DDA4D: G***, kibuzzard-631DDA4D, F.Cu at (103.5, 101.5)
- added kibuzzard-63351CB9: G***, kibuzzard-63351CB9, F.Cu at (102.5, 118.5)
Routing:
- added copper zone on B.Cu, net (none)
- added copper zone on F.Cu, net (none)
- removed copper zone on B.Cu, net GND
- removed copper zone on F.Cu, net GND
Other:
- board size 42.1 x 24.6 mm -> 39.6 x 19.6 mm
- board text added: "TEMPLATE"
